File: master.brd (EAGLE design)
At the start: 160 x 120 mm, 318 parts, among them IC1001 AQV252G2S, IC1002 AQV252G2S, IC1003 AQV252G2S, IC1004 AQV252G2S, IC1005 AQV252G2S, IC1006 AQV252G2S, IC1101 UA78L05ACPK, IC1102 ADUM3300ARW, IC1103 ADUM3300ARW, IC1401 IP4220CZ6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

Commit message: fixed fuse value in schematic
Parts:
- F1001, F1002, F1003, F1004, F1005, F1006: value 630MA_UMT -> 4,00A_UMT
